Commit message: v2.0 (new race-track and multiple racecars)

File: urdf/macros.xacro (robot description, xacro)
@@ -44,5 +44,5 @@
     <origin xyz="0.46 -0.135 -0.180" rpy="1.57 0 3.14" />
     <geometry>
-      <mesh filename="package://f1tenth-sim/urdf/meshes/chassis.stl" scale="0.000990 0.0009375 0.0009375"/>
+      <mesh filename="package://spring_2020_virtual_class/urdf/meshes/chassis.stl" scale="0.000990 0.0009375 0.0009375"/>
     </geometry>
   </xacro:macro>
@@ -50,5 +50,5 @@
     <origin xyz="0 0 0" rpy="0 0 0" />
     <geometry>
-      <mesh filename="package://f1tenth-sim/urdf/meshes/left_wheel.stl" />
+      <mesh filename="package://spring_2020_virtual_class/urdf/meshes/left_wheel.stl" />
     </geometry>
   </xacro:macro>
@@ -56,5 +56,5 @@
     <origin xyz="0 0 0" rpy="0 0 0" />
     <geometry>
-      <mesh filename="package://f1tenth-sim/urdf/meshes/right_wheel.stl" />
+      <mesh filename="package://spring_2020_virtual_class/urdf/meshes/right_wheel.stl" />
     </geometry>
   </xacro:macro>
@@ -62,5 +62,5 @@
     <origin xyz="0 0 0" rpy="0 0 0" />
     <geometry>
-      <mesh filename="package://f1tenth-sim/urdf/meshes/left_wheel.stl" />
+      <mesh filename="package://spring_2020_virtual_class/urdf/meshes/left_wheel.stl" />
     </geometry>
   </xacro:macro>
@@ -68,5 +68,5 @@
     <origin xyz="0 0 0" rpy="0 0 0" />
     <geometry>
-      <mesh filename="package://f1tenth-sim/urdf/meshes/right_wheel.stl" />
+      <mesh filename="package://spring_2020_virtual_class/urdf/meshes/right_wheel.stl" />
     </geometry>
   </xacro:macro>
@@ -74,5 +74,5 @@
     <origin xyz="0 0 0" rpy="0 0 0" />
     <geometry>
-      <mesh filename="package://f1tenth-sim/urdf/meshes/hinge.stl" />
+      <mesh filename="package://spring_2020_virtual_class/urdf/meshes/hinge.stl" />
     </geometry>
   </xacro:macro>
@@ -80,5 +80,5 @@
     <origin xyz="0 0 0" rpy="0 0 0" />
     <geometry>
-      <mesh filename="package://f1tenth-sim/urdf/meshes/hinge.stl" />
+      <mesh filename="package://spring_2020_virtual_class/urdf/meshes/hinge.stl" />
     </geometry>
   </xacro:macro>
@@ -277,5 +277,5 @@
       <origin xyz="0 0 0" rpy="0 0 0"/>
       <geometry>
-        <mesh filename="package://f1tenth-sim/urdf/meshes/hokuyo.stl"/>
+        <mesh filename="package://spring_2020_virtual_class/urdf/meshes/hokuyo.stl"/>
         <material name="grey" />
       </geometry>
@@ -320,5 +320,5 @@
     <inertial>
       <mass value="1e-5" />
-      <origin xyz="-0.25 0 0.025" rpy="0 0 0"/>
+      <origin xyz="-2.5 1.5 1.75" rpy="0 .57 -0.57"/>
       <inertia ixx="1e-6" ixy="0" ixz="0" iyy="1e-6" iyz="0" izz="1e-6" />
     </inertial>
@@ -327,10 +327,10 @@
     <inertial>
       <mass value="1e-5" />
-      <origin xyz="0 0 0.025" rpy="0 0 0"/>
+      <origin xyz="-2.5 1.5 1.75" rpy="0 .57 -0.57"/>
       <inertia ixx="1e-6" ixy="0" ixz="0" iyy="1e-6" iyz="0" izz="1e-6" />
     </inertial>
   </link>
   <joint name="$(arg robot_name)_left_joint" type="fixed">
-    <origin xyz="0 0 0.035" rpy="0 0 0"/>
+    <origin xyz="-2.5 1.5 1.75" rpy="0 .57 -0.57"/>
     <parent link="$(arg robot_name)_link"/>
     <child link="$(arg robot_name)_camera_link"/>

Commit message: Fixed path issues

File: urdf/macros.xacro (robot description, xacro)
@@ -44,5 +44,5 @@
     <origin xyz="0.46 -0.135 -0.180" rpy="1.57 0 3.14" />
     <geometry>
-      <mesh filename="package://spring_2020_virtual_class/urdf/meshes/chassis.stl" scale="0.000990 0.0009375 0.0009375"/>
+      <mesh filename="package://f1tenth-sim/urdf/meshes/chassis.stl" scale="0.000990 0.0009375 0.0009375"/>
     </geometry>
   </xacro:macro>
@@ -50,5 +50,5 @@
     <origin xyz="0 0 0" rpy="0 0 0" />
     <geometry>
-      <mesh filename="package://spring_2020_virtual_class/urdf/meshes/left_wheel.stl" />
+      <mesh filename="package://f1tenth-sim/urdf/meshes/left_wheel.stl" />
     </geometry>
   </xacro:macro>
@@ -56,5 +56,5 @@
     <origin xyz="0 0 0" rpy="0 0 0" />
     <geometry>
-      <mesh filename="package://spring_2020_virtual_class/urdf/meshes/right_wheel.stl" />
+      <mesh filename="package://f1tenth-sim/urdf/meshes/right_wheel.stl" />
     </geometry>
   </xacro:macro>
@@ -62,5 +62,5 @@
     <origin xyz="0 0 0" rpy="0 0 0" />
     <geometry>
-      <mesh filename="package://spring_2020_virtual_class/urdf/meshes/left_wheel.stl" />
+      <mesh filename="package://f1tenth-sim/urdf/meshes/left_wheel.stl" />
     </geometry>
   </xacro:macro>
@@ -68,5 +68,5 @@
     <origin xyz="0 0 0" rpy="0 0 0" />
     <geometry>
-      <mesh filename="package://spring_2020_virtual_class/urdf/meshes/right_wheel.stl" />
+      <mesh filename="package://f1tenth-sim/urdf/meshes/right_wheel.stl" />
     </geometry>
   </xacro:macro>
@@ -74,5 +74,5 @@
     <origin xyz="0 0 0" rpy="0 0 0" />
     <geometry>
-      <mesh filename="package://spring_2020_virtual_class/urdf/meshes/hinge.stl" />
+      <mesh filename="package://f1tenth-sim/urdf/meshes/hinge.stl" />
     </geometry>
   </xacro:macro>
@@ -80,5 +80,5 @@
     <origin xyz="0 0 0" rpy="0 0 0" />
     <geometry>
-      <mesh filename="package://spring_2020_virtual_class/urdf/meshes/hinge.stl" />
+      <mesh filename="package://f1tenth-sim/urdf/meshes/hinge.stl" />
     </geometry>
   </xacro:macro>
@@ -277,5 +277,5 @@
       <origin xyz="0 0 0" rpy="0 0 0"/>
       <geometry>
-        <mesh filename="package://spring_2020_virtual_class/urdf/meshes/hokuyo.stl"/>
+        <mesh filename="package://f1tenth-sim/urdf/meshes/hokuyo.stl"/>
         <material name="grey" />
       </geometry>

Commit message: New dissertation setup

File: urdf/macros.xacro (robot description, xacro)
@@ -213,5 +213,5 @@
     </visual>
   </link>
-  <joint name="$(arg robot_name)_right_steering_hinge_joint" type="continuous">
+  <joint name="$(arg robot_name)_right_steering_hinge_joint" type="revolute">
     <origin xyz="0.325 -0.1 0" rpy="0 1.5708 0" />
     <parent link="$(arg robot_name)_chassis" />
@@ -320,5 +320,5 @@
     <inertial>
       <mass value="1e-5" />
-      <origin xyz="-2.5 1.5 1.75" rpy="0 .57 -0.57"/>
+      <origin xyz="-2.5 0 1.75" rpy="0 .57 0"/>
       <inertia ixx="1e-6" ixy="0" ixz="0" iyy="1e-6" iyz="0" izz="1e-6" />
     </inertial>
@@ -327,10 +327,10 @@
     <inertial>
       <mass value="1e-5" />
-      <origin xyz="-2.5 1.5 1.75" rpy="0 .57 -0.57"/>
+      <origin xyz="-2.5 0 1.75" rpy="0 .57 0"/>
       <inertia ixx="1e-6" ixy="0" ixz="0" iyy="1e-6" iyz="0" izz="1e-6" />
     </inertial>
   </link>
   <joint name="$(arg robot_name)_left_joint" type="fixed">
-    <origin xyz="-2.5 1.5 1.75" rpy="0 .57 -0.57"/>
+    <origin xyz="-2.5 0 1.75" rpy="0 .57 0"/>
     <parent link="$(arg robot_name)_link"/>
     <child link="$(arg robot_name)_camera_link"/>
@@ -430,5 +430,5 @@
           </noise>
         </ray>
-        <plugin name="gazebo_ros_hokuyo_controller" filename="libgazebo_ros_laser.so">
+        <plugin name="hokuyo_controller" filename="libgazebo_ros_laser.so">
           <topicName>/$(arg robot_name)/scan</topicName>
           <frameName>$(arg robot_name)_laser</frameName>

Commit message: refactor and organize codes

File: urdf/macros.xacro (robot description, xacro)
@@ -127,4 +127,7 @@
       <material name="red" />
     </visual>
+    <collision>
+      <xacro:chassis_geometry />
+    </collision>
   </link>
   <joint name="$(arg robot_name)_base_link_joint" type="fixed">
@@ -152,5 +155,5 @@
       <material name="black" />
     </visual>
-    <collision>robot
+    <collision>
       <xacro:left_wheels_collision_geometry />
     </collision>

Commit message: fix laser tf, update launchfile

File: urdf/macros.xacro (robot description, xacro)
@@ -272,5 +272,5 @@
     </inertial>
     <collision>
-      <origin xyz="0 0 0" rpy="0 0 0"/>
+      <origin xyz="0 0 -0.018" rpy="0 0 0"/>
       <geometry>
         <box size="0.1 0.1 0.1"/>
@@ -278,5 +278,5 @@
     </collision>
     <visual>
-      <origin xyz="0 0 0" rpy="0 0 0"/>
+      <origin xyz="0 0 -0.018" rpy="0 0 0"/>
       <geometry>
         <mesh filename="package://f1tenth-sim/urdf/meshes/hokuyo.stl"/>
@@ -286,5 +286,5 @@
   </link>
   <joint name="$(arg robot_name)_hokuyo_joint" type="fixed">
-    <origin xyz="0.125 0.0 0.155" rpy="0 0 0"/>
+    <origin xyz="0.125 0.0 0.173" rpy="0 0 0"/>
     <parent link="$(arg robot_name)_chassis" />
     <child link="$(arg robot_name)_laser" />
@@ -406,10 +406,10 @@
     </plugin>
   </gazebo>
-    <!-- hokuyo -->
+  <!-- hokuyo -->
   <xacro:unless value="$(optenv DISABLE_GAZEBO_LASER false)">
     <gazebo reference="$(arg robot_name)_laser">
       <material>Gazebo/Grey</material>
       <sensor type="ray" name="$(arg robot_name)_hokuyo_sensor">
-        <pose>0 0 0.0124 0 0 0</pose>
+        <pose>0 0 0 0 0 0</pose>
         <visualize>false</visualize>
         <update_rate>40</update_rate>
